File: hw/FreshTwinkie_v0.1/FreshTwinkie.sch (KiCad schematic (older format))
At the start: 54 parts, among them J1 USB_C_Receptacle, J2 USB_B_Micro, P1 USB_C_Plug, Q1 BSD840NH6327XTSA1, Q2 BSD840NH6327XTSA1, Q3 BSD840NH6327XTSA1, Q4 BSD840NH6327XTSA1, SW1 SW_Push, U1 AD8606ARMZ-REEL, U2 STM32F072CBUx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

Commit message: changeLanguagesch
Other:
- note added: "Bootloader Mode\n"
- note added: "Leds \n\n\n"
- note added: "Micro-B y voltage regulator"
- note added: "To enter in bootmode, plug in A-to-A cable trought \nOGT adaptador. Or use an micro-B while plug in, push SW1. \n"
- note removed: "Leds indicadores\n\n"
- note removed: "Micro-B y regulador de voltaje\n\n"
- note removed: "Modo Bootloader\n"
- note removed: "Para entrar en el modo boot, \nconectar un cable A-to-A en un adaptador OGT \no usar un cable Micro-B y mientrás se inserta, \npresionar el SW1."
Changed lines of the file:
@@
 BOOT
 Text Notes 15500 6550 2    197  ~ 0
-Modo Bootloader\n
+Bootloader Mode\n
 Text Label 5650 2250 0    50   ~ 0
 CC1_BUF
@@
 Wire Wire Line
 	14700 9350 14750 9350
-Text Notes 12950 7100 0    79   ~ 0
-Para entrar en el modo boot, \nconectar un cable A-to-A en un adaptador OGT \no usar un cable Micro-B y mientrás se inserta, \npresionar el SW1.
+Text Notes 12850 6850 0    63   ~ 0
+To enter in bootmode, plug in A-to-A cable trought \nOGT adaptador. Or use an micro-B while plug in, push SW1. \n
 Text Label 13800 8500 2    50   ~ 0
 USB_B_ID
@@
 	8800 1500 8800 2000
 Text Notes 8300 1300 0    197  ~ 0
-Leds indicadores\n\n
+Leds \n\n\n
 Wire Notes Line
 	8000 3450 11200 3450
@@
 	4650 8550 4650 8450
 Text Notes 5650 7450 2    197  ~ 0
-Micro-B y regulador de voltaje\n\n
+Micro-B y voltage regulator
 Text Label 14450 5300 0    50   ~ 0
 CC1_RPUSB

Commit message: changeNameProjectshc
Other:
- note added: "To enter in bootmode, plug in A-to-A cable trought \nOGT adaptador. Or use a micro-B cable, while plug in push SW1. \n"
- note removed: "To enter in bootmode, plug in A-to-A cable trought \nOGT adaptador. Or use an micro-B while plug in, push SW1. \n"
Changed lines of the file:
@@
 encoding utf-8
 Sheet 1 1
-Title "ClockClock Module"
-Date "2019-03-23"
+Title "USBC-PDSniffer"
+Date "2021-03-16"
 Rev "r0_1"
-Comp "GsD"
+Comp "Electronic Cats"
 Comment1 ""
 Comment2 ""
@@
 Wire Wire Line
 	14700 9350 14750 9350
-Text Notes 12850 6850 0    63   ~ 0
-To enter in bootmode, plug in A-to-A cable trought \nOGT adaptador. Or use an micro-B while plug in, push SW1. \n
+Text Notes 11950 6850 0    79   ~ 0
+To enter in bootmode, plug in A-to-A cable trought \nOGT adaptador. Or use a micro-B cable, while plug in push SW1. \n
 Text Label 13800 8500 2    50   ~ 0
 USB_B_ID
@@
 	13800 8500 14150 8500
 Wire Notes Line
-	12800 6200 12800 9900
-Wire Notes Line
-	12800 9900 16050 9900
+	11900 6250 11900 9950
 $Comp
 L power:+3.3V #PWR04

Commit message: correctComponentsPN
Parts:
- C1, C6: Mfg Murata -> Samsung; PN C77004 -> C1705
- C2, C3, C7: Mfg YAGEO -> Samsung; PN C60474 -> C1591
- C4: Mfg YAGEO -> Samsung; PN C272878 -> C1589
- C5, C8, C9: PN C307454 -> C29936
- R1, R12: PN C325381 -> C269905
- R10, R9: Mfg Viking Tech -> TyoHM; PN C284520 -> C269375
- R11: Mfg ROHM Semicon -> TyoHM; PN C525583 -> C325718
- R13, R18, R2, R22, R23, R5: PN C284526 -> C217980
- R14, R15, R16, R3: Mfg YAGEO -> Viking Tech; PN C723406 -> C374574
- R17, R4: Mfg YAGEO -> Viking Tech; PN C281773 -> C217717
- R19, R6: Mfg Viking Tech -> Vishay; PN C317916 -> C161809
- R20, R7: PN C274895 -> C706183
- R21, R24, R8: PN C325391 -> C269683

Commit message: chngComponentOOS
Parts:
- U3: PN 621-AP2112K-3.3TRG1 -> C51118; Tienda Mouser -> LCSC
Changed lines of the file:
@@
 F 1 "AP2112K" H 4650 8426 50  0000 C CNN
 F 2 "Package_TO_SOT_SMD:SOT-23-5" H 4650 7750 50  0001 C CNN
-F 3 "https://www.mouser.mx/datasheet/2/115/AP2112-271550.pdf" H 4400 8400 50  0001 C CNN
+F 3 "https://datasheet.lcsc.com/szlcsc/1809192242_Diodes-Incorporated-AP2112K-3-3TRG1_C51118.pdf" H 4400 8400 50  0001 C CNN
 F 4 "Diodes Incorporated" H 4650 8150 50  0001 C CNN "Mfg"
-F 5 "621-AP2112K-3.3TRG1" H 4650 8150 50  0001 C CNN "PN"
-F 6 "Mouser" H 4650 8150 50  0001 C CNN "Tienda"
+F 5 "C51118" H 4650 8150 50  0001 C CNN "PN"
+F 6 "LCSC" H 4650 8150 50  0001 C CNN "Tienda"
 	1    4650 8150
 	1    0    0    -1
